File: tomu-eagle0.brd (EAGLE design)
At the start: 14.4 x 9.7 mm, 18 parts, among them U1 EFM32HG309F64G

Commit message: LED resistors should be 75 not 15 (or maybe 52 as in the tomu bom)
Parts:
- R1, R2: value 15 -> 75
Changed lines of the file:
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@@
 <?xml version="1.0" encoding="utf-8"?>
 <!DOCTYPE eagle SYSTEM "eagle.dtd">
-<eagle version="8.6.0">
+<eagle version="8.7.1">
 <drawing>
 <settings>
@@
 <attribute name="VALUE" x="10.414" y="11.303" size="1.27" layer="28" rot="MR180"/>
 </element>
-<element name="R1" library="adafruit" library_urn="urn:adsk.eagle:library:420" package="R0402" value="15" x="11.049" y="8.382" smashed="yes" rot="MR0">
+<element name="R1" library="adafruit" library_urn="urn:adsk.eagle:library:420" package="R0402" value="75" x="11.049" y="8.382" smashed="yes" rot="MR0">
 <attribute name="NAME" x="10.541" y="7.874" size="0.6096" layer="26" ratio="12" rot="MR180"/>
 <attribute name="VALUE" x="11.684" y="6.35" size="1.27" layer="28" rot="MR0"/>
 </element>
-<element name="R2" library="adafruit" library_urn="urn:adsk.eagle:library:420" package="R0402" value="15" x="11.049" y="3.302" smashed="yes" rot="MR0">
+<element name="R2" library="adafruit" library_urn="urn:adsk.eagle:library:420" package="R0402" value="75" x="11.049" y="3.302" smashed="yes" rot="MR0">
 <attribute name="NAME" x="11.557" y="3.81" size="0.6096" layer="26" ratio="12" rot="MR0"/>
 </element>
