File: tomu-pro-micro.brd (EAGLE design)
At the start: 29.7 x 16 mm, 15 parts, among them SW1 SPST_TACT-KMR2, U1 EFM32HG309F64G

Commit message: LED resistors should be 75 not 15 (or maybe 52 as in the tomu bom)
Parts:
- R1, R2: value 15 -> 75
Changed lines of the file:
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@@
 <attribute name="VALUE" x="12.7" y="8.255" size="1.27" layer="27" rot="R180"/>
 </element>
-<element name="R1" library="adafruit" library_urn="urn:adsk.eagle:library:420" package="R0603" value="15" x="-6.223" y="2.286" smashed="yes">
+<element name="R1" library="adafruit" library_urn="urn:adsk.eagle:library:420" package="R0603" value="75" x="-6.223" y="2.286" smashed="yes">
 <attribute name="NAME" x="-5.715" y="1.524" size="0.6096" layer="25" ratio="12" rot="R180"/>
 <attribute name="VALUE" x="-6.858" y="0.254" size="1.27" layer="27"/>
 </element>
-<element name="R2" library="adafruit" library_urn="urn:adsk.eagle:library:420" package="R0603" value="15" x="-6.223" y="-1.778" smashed="yes">
+<element name="R2" library="adafruit" library_urn="urn:adsk.eagle:library:420" package="R0603" value="75" x="-6.223" y="-1.778" smashed="yes">
 <attribute name="NAME" x="-6.477" y="-1.016" size="0.6096" layer="25" ratio="12"/>
 <attribute name="VALUE" x="-6.858" y="-3.81" size="1.27" layer="27"/>
