File: tomu-pro-micro2.brd (EAGLE design)
At the start: 32 x 18 mm, 19 parts, among them SW1 SPST_TACT-KMR2, U1 EFM32HG309F64G

Commit message: fix problems with tomo-pro-micro1
Connections:
- removed net V+: C4.1, D1.A, L2.2
- net VUSB: now also C4.1, D1.A, L2.2
Routing:
- net VUSB: track 19.6 -> 43.3 mm, vias 2 -> 3
- net V+: track 5.03 -> 0.00 mm
- net GND: track 13.1 -> 13.7 mm
Other:
- board text added: "20180527"
- board text added: "tomu-pro-micro2"
- board text removed: "20180421"
- board text removed: "tomu-pro-micro1"
