File: tomu-pro-micro2.sch (EAGLE design)
At the start: 19 parts, among them SW1 SPST_TACT-KMR2, U1 EFM32HG309F64G

Commit message: fix problems with tomo-pro-micro1
Connections:
- removed net V+: C4.1, D1.A, L2.VDD
- net VUSB: now also C4.1, D1.A, L2.VDD
Changed lines of the file:
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@@
 <part name="L1" library="todstuff" library_urn="urn:adsk.eagle:library:1731349" deviceset="WS2812B" device="3535" package3d_urn="urn:adsk.eagle:package:1731511/1"/>
 <part name="GND6" library="supply1" library_urn="urn:adsk.eagle:library:371" deviceset="GND" device=""/>
-<part name="VBUS3" library="supply1" library_urn="urn:adsk.eagle:library:371" deviceset="V+" device=""/>
 <part name="L2" library="todstuff" library_urn="urn:adsk.eagle:library:1731349" deviceset="WS2812B" device="3535" package3d_urn="urn:adsk.eagle:package:1731511/1"/>
 <part name="GND7" library="supply1" library_urn="urn:adsk.eagle:library:371" deviceset="GND" device=""/>
@@
 <part name="VBUS5" library="supply1" library_urn="urn:adsk.eagle:library:371" deviceset="V+" device=""/>
 <part name="U1" library="todstuff" library_urn="urn:adsk.eagle:library:1731349" deviceset="EFM32HG309F64G" device="" package3d_urn="urn:adsk.eagle:package:1731515/8"/>
+<part name="VBUS6" library="supply1" library_urn="urn:adsk.eagle:library:371" deviceset="V+" device=""/>
 </parts>
 <sheets>
@@
 <instance part="L1" gate="G$1" x="124.46" y="124.46"/>
 <instance part="GND6" gate="1" x="124.46" y="111.76"/>
-<instance part="VBUS3" gate="1" x="114.3" y="147.32"/>
 <instance part="L2" gate="G$1" x="149.86" y="124.46"/>
 <instance part="GND7" gate="1" x="149.86" y="111.76"/>
@@
 <instance part="VBUS5" gate="1" x="139.7" y="157.48"/>
 <instance part="U1" gate="G$1" x="71.12" y="53.34"/>
+<instance part="VBUS6" gate="1" x="104.14" y="147.32"/>
 </instances>
 <busses>
@@
 <wire x1="50.8" y1="144.78" x2="73.66" y2="144.78" width="0.1524" layer="91"/>
 <label x="58.42" y="144.78" size="1.778" layer="95"/>
+</segment>
+<segment>
+<pinref part="L2" gate="G$1" pin="VDD"/>
+<pinref part="VBUS4" gate="1" pin="V+"/>
+<wire x1="154.94" y1="139.7" x2="154.94" y2="144.78" width="0.1524" layer="91"/>
+</segment>
+<segment>
+<pinref part="D1" gate="G$1" pin="A"/>
+<pinref part="VBUS6" gate="1" pin="V+"/>
+<wire x1="119.38" y1="142.24" x2="104.14" y2="142.24" width="0.1524" layer="91"/>
+<wire x1="104.14" y1="142.24" x2="104.14" y2="144.78" width="0.1524" layer="91"/>
+<label x="106.68" y="142.24" size="1.778" layer="95"/>
+</segment>
+<segment>
+<pinref part="C4" gate="G$1" pin="1"/>
+<pinref part="VBUS5" gate="1" pin="V+"/>
 </segment>
 </net>
@@
 </segment>
 </net>
-<net name="V+" class="0">
-<segment>
-<pinref part="L2" gate="G$1" pin="VDD"/>
-<pinref part="VBUS4" gate="1" pin="V+"/>
-<wire x1="154.94" y1="139.7" x2="154.94" y2="144.78" width="0.1524" layer="91"/>
-</segment>
-<segment>
-<pinref part="D1" gate="G$1" pin="A"/>
-<pinref part="VBUS3" gate="1" pin="V+"/>
-<wire x1="119.38" y1="142.24" x2="114.3" y2="142.24" width="0.1524" layer="91"/>
-<wire x1="114.3" y1="142.24" x2="114.3" y2="144.78" width="0.1524" layer="91"/>
-</segment>
-<segment>
-<pinref part="C4" gate="G$1" pin="1"/>
-<pinref part="VBUS5" gate="1" pin="V+"/>
-</segment>
-</net>
